File: Single-Sided 5V Power Supply.kicad_sch (KiCad schematic)
At the start: 7 parts, among them J1 9V AC INPUT, J2 +5V OUTPUT, U1 L7805

Commit message: Update capacitor values based on LM7805 datasheet recommendations
Parts:
- C1: value 470u -> 3300uF
- C2: value 0.01u -> 0.33uF
- C3: value 0.01u -> 0.01uF
Changed lines of the file:
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@@
 			)
 		)
-		(property "Value" "470u"
+		(property "Value" "3300uF"
 			(at 149.86 80.3909 0)
 			(effects
@@
 			)
 		)
-		(property "Value" "0.01u"
+		(property "Value" "0.33uF"
 			(at 166.37 81.2799 0)
 			(effects
@@
 			)
 		)
-		(property "Value" "0.01u"
+		(property "Value" "0.01uF"
 			(at 182.88 81.2799 0)
 			(effects
